File: Powery.kicad_pcb (KiCad board)
At the start: 2 copper layers, 0 parts

Commit message: WIP layout.
Parts:
- added C101: 10uf, Capacitors_SMD:C_0805_HandSoldering, F.Cu at (282.1, 67.9)
- added C102: 4.7uf, Capacitors_SMD:C_0805_HandSoldering, F.Cu at (262.8, 84.9)
- added C103: 100nf, Capacitors_SMD:C_0805_HandSoldering, F.Cu at (267.5, 72.2)
- added C104: 100nf, Capacitors_SMD:C_0805_HandSoldering, F.Cu at (270.5, 78.6)
- added C105: 100nf, Capacitors_SMD:C_0805, F.Cu at (261.2, 78.6)
- added C106: 100nf, Capacitors_SMD:C_0805, F.Cu at (248.1, 96.2)
- added C107: 100nf, Capacitors_SMD:C_0805, F.Cu at (276.8, 71.9)
- added C108: 10nf, Capacitors_SMD:C_0805, F.Cu at (272.2, 71.9)
- added C109: 1uf, Capacitors_SMD:C_0805, F.Cu at (265.8, 78.6)
- added C110: 20pf, Capacitors_SMD:C_0805, F.Cu at (258.0, 85.5)
- added C111: 20pf, Capacitors_SMD:C_0805, F.Cu at (281.7, 61.5)
- added C201: NP, Capacitors_SMD:C_0805, F.Cu at (133.1, 61.5)
- added C202: 0.1u, Capacitors_SMD:C_0805, F.Cu at (161.9, 68.8)
- added C203: 0.1u, Capacitors_SMD:C_0805, F.Cu at (149.9, 49.3)
- added C204: 0.1u, Capacitors_SMD:C_0805, F.Cu at (157.0, 64.5)
- added C205: 0.1u, Capacitors_SMD:C_0805, F.Cu at (154.9, 51.3)
- added C206: 1uf, Capacitors_SMD:C_0805, F.Cu at (91.4, 65.0)
- added C207: 10uf, Capacitors_SMD:C_0805, B.Cu at (157.5, 57.9)
- added C208: 10uf, Capacitors_SMD:C_0805, B.Cu at (138.7, 70.3)
- added C209: 10uf, Capacitors_SMD:C_0805, F.Cu at (130.6, 79.8)
- added C301: NP, Capacitors_SMD:C_0805, F.Cu at (193.1, 121.5)
- added C302: 0.1u, Capacitors_SMD:C_0805, F.Cu at (198.5, 115.1)
- added C303: 0.1u, Capacitors_SMD:C_0805, F.Cu at (192.3, 108.8)
- added C304: 0.1u, Capacitors_SMD:C_0805, F.Cu at (165.1, 134.8)
- added C305: 0.1u, Capacitors_SMD:C_0805, F.Cu at (202.8, 115.1)
- added C306: 1uf, Capacitors_SMD:C_0805, F.Cu at (88.4, 64.0)
- added C307: 10uf, Capacitors_SMD:C_0805, F.Cu at (186.9, 131.3)
- added C308: 10uf, Capacitors_SMD:C_0805, F.Cu at (170.4, 146.2)
- added C309: 10uf, Capacitors_SMD:C_0805, F.Cu at (207.2, 115.1)
- added CON101: BARREL_JACK, Connect:JACK_ALIM, F.Cu at (64.0, 84.8)
- added D201: D, TO_SOT_Packages_SMD:SOT-23_Handsoldering, F.Cu at (128.5, 72.6)
- added D202: D, Diodes_SMD:SMA-SMB_Universal_Handsoldering, F.Cu at (126.0, 81.8)
- added D301: D, TO_SOT_Packages_SMD:SOT-23_Handsoldering, F.Cu at (185.2, 110.5)
- added D302: D, Diodes_SMD:SMA-SMB_Universal_Handsoldering, F.Cu at (84.0, 68.6)
- added HS201: HEATSINK, gl:HS-TO220-20W, F.Cu at (109.7, 60.5)
- added HS301: HEATSINK, gl:HS-TO220-20W, F.Cu at (109.7, 103.1)
- added JP101: Jumper_NO_Small, stmps:MADW__SMD-solder-bridge-narrow, F.Cu at (224.7, 75.2)
- added K201: RELAY-SPDT, gl:RELAY-SRD, F.Cu at (133.1, 47.2)
- added K301: RELAY-SPDT, gl:RELAY-SRD, F.Cu at (170.2, 113.9)
- added P101: CONN_01X02, Pin_Headers:Pin_Header_Straight_1x02, F.Cu at (274.6, 60.7)
- added P102: CONN_01X03, Pin_Headers:Pin_Header_Straight_1x03, F.Cu at (242.0, 64.5)
- added P103: CONN_01X02, Pin_Headers:Pin_Header_Straight_1x02, F.Cu at (215.6, 64.5)
- added P104: CONN_01X03, Pin_Headers:Pin_Header_Straight_1x03, F.Cu at (215.6, 85.4)
- added P105: CONN_01X02, Pin_Headers:Pin_Header_Straight_1x02, F.Cu at (250.8, 88.5)
- added P106: USB_OTG, stmps:USB_Micro-B-ebay, F.Cu at (230.4, 84.2)
- added P107: LCD1, Pin_Headers:Pin_Header_Straight_1x06, F.Cu at (264.6, 64.5)
- added P108: LCD2, Pin_Headers:Pin_Header_Straight_1x06, F.Cu at (240.6, 82.9)
- added P109: CONN_01X06, Pin_Headers:Pin_Header_Straight_1x05, F.Cu at (240.6, 96.1)
- added P110: CONN_01X02, Wire_Connections_Bridges:WireConnection_2.50mmDrill, F.Cu at (146.8, 103.1)
- added P111: CONN_01X02, Wire_Connections_Bridges:WireConnection_2.50mmDrill, F.Cu at (147.3, 43.2)
- added Q201: MMBT3904, TO_SOT_Packages_SMD:SOT-23, F.Cu at (145.9, 60.7)
- added Q202: MMBT3904, TO_SOT_Packages_SMD:SOT-23, F.Cu at (145.4, 50.8)
- added Q203: MMBT3904, TO_SOT_Packages_SMD:SOT-23, F.Cu at (126.0, 56.9)
- added Q301: MMBT3904, TO_SOT_Packages_SMD:SOT-23, F.Cu at (158.7, 137.7)
- added Q302: MMBT3904, TO_SOT_Packages_SMD:SOT-23, F.Cu at (175.2, 127.0)
- added Q303: MMBT3904, TO_SOT_Packages_SMD:SOT-23, F.Cu at (156.7, 145.2)
- added R101: 2.2k, Resistors_SMD:R_0805_HandSoldering, F.Cu at (281.1, 80.6)
- added R102: 2.2k, Resistors_SMD:R_0805_HandSoldering, F.Cu at (262.2, 72.2)
- added R103: 4.7k, Resistors_SMD:R_0805_HandSoldering, F.Cu at (263.9, 91.3)
- added R104: 10k, Resistors_SMD:R_0805_HandSoldering, F.Cu at (281.9, 74.2)
- added R105: 220, Resistors_SMD:R_0805_HandSoldering, F.Cu at (268.0, 84.9)
- added R106: 4.3k, Resistors_SMD:R_0805_HandSoldering, F.Cu at (275.8, 78.3)
- added R107: 4.3k, Resistors_SMD:R_0805_HandSoldering, F.Cu at (275.8, 84.6)
- added R108: 10k, Resistors_SMD:R_0805_HandSoldering, F.Cu at (286.5, 61.5)
- added R109: 10k, Resistors_SMD:R_0805_HandSoldering, F.Cu at (258.5, 91.8)
- added R201: 0, Resistors_SMD:R_0805_HandSoldering, F.Cu at (125.5, 67.6)
- added R202: 0, Resistors_SMD:R_0805_HandSoldering, F.Cu at (149.9, 51.3)
- added R203: 100k, Resistors_SMD:R_0805_HandSoldering, F.Cu at (167.6, 64.5)
- added R204: 100k, Resistors_SMD:R_0805_HandSoldering, F.Cu at (154.9, 49.3)
- added R205: 0.22, Resistors_SMD:R_2512_HandSoldering, F.Cu at (140.7, 62.0)
- added R206: 0.22, Resistors_SMD:R_2512_HandSoldering, F.Cu at (136.7, 62.0)
- added R207: 100k, Resistors_SMD:R_0805_HandSoldering, F.Cu at (157.0, 66.5)
- added R208: 100k, Resistors_SMD:R_0805_HandSoldering, F.Cu at (131.1, 59.1)
- added R209: 10k, Resistors_SMD:R_0805_HandSoldering, F.Cu at (162.1, 66.5)
- added R210: 100k, Resistors_SMD:R_0805_HandSoldering, F.Cu at (162.1, 64.5)
- added R211: 4.3k, Resistors_SMD:R_0805_HandSoldering, F.Cu at (160.0, 57.9)
- added R212: 10k, Resistors_SMD:R_0805_HandSoldering, F.Cu at (145.3, 66.2)
- added R213: 100k, Resistors_SMD:R_0805_HandSoldering, F.Cu at (147.3, 66.0)
- added R214: 10k, Resistors_SMD:R_0805_HandSoldering, F.Cu at (157.5, 71.6)
- added R215: 10k, Resistors_SMD:R_0805_HandSoldering, F.Cu at (87.0, 61.5)
- added R216: 10k, Resistors_SMD:R_0805_HandSoldering, F.Cu at (151.4, 66.5)
- added R217: 1k, Resistors_SMD:R_0805_HandSoldering, F.Cu at (151.4, 64.5)
- added R218: 100, Resistors_SMD:R_0805_HandSoldering, F.Cu at (147.0, 56.4)
- added R219: 1k, Resistors_SMD:R_0805_HandSoldering, F.Cu at (144.5, 56.4)
- added R220: 10k, Resistors_SMD:R_0805_HandSoldering, F.Cu at (151.4, 69.1)
- added R221: 100, Resistors_SMD:R_0805_HandSoldering, F.Cu at (141.7, 75.2)
- added R301: 0, Resistors_SMD:R_0805_HandSoldering, F.Cu at (173.7, 133.5)
- added R302: 0, Resistors_SMD:R_0805_HandSoldering, F.Cu at (165.6, 141.2)
- added R303: 100k, Resistors_SMD:R_0805_HandSoldering, F.Cu at (176.3, 139.9)
- added R304: 100k, Resistors_SMD:R_0805_HandSoldering, F.Cu at (188.3, 118.6)
- added R305: 0.22, Resistors_SMD:R_2512_HandSoldering, F.Cu at (133.5, 126.8)
- added R306: 0.22, Resistors_SMD:R_2512_HandSoldering, F.Cu at (133.5, 112.4)
- added R307: 100k, Resistors_SMD:R_0805_HandSoldering, F.Cu at (182.0, 126.8)
- added R308: 100k, Resistors_SMD:R_0805_HandSoldering, F.Cu at (170.9, 139.9)
- added R309: 10k, Resistors_SMD:R_0805_HandSoldering, F.Cu at (193.6, 115.1)
- added R310: 100k, Resistors_SMD:R_0805_HandSoldering, F.Cu at (187.4, 124.9)
- added R311: 4.3k, Resistors_SMD:R_0805_HandSoldering, F.Cu at (202.5, 108.8)
- added R312: 10k, Resistors_SMD:R_0805_HandSoldering, F.Cu at (197.2, 108.8)
- added R313: 100k, Resistors_SMD:R_0805_HandSoldering, F.Cu at (182.9, 118.6)
- added R314: 10k, Resistors_SMD:R_0805_HandSoldering, F.Cu at (192.3, 134.2)
- added R315: 10k, Resistors_SMD:R_0805_HandSoldering, F.Cu at (79.9, 62.0)
- added R316: 10k, Resistors_SMD:R_0805_HandSoldering, F.Cu at (203.3, 121.5)
- added R317: 1k, Resistors_SMD:R_0805_HandSoldering, F.Cu at (179.0, 133.5)
- added R318: 100, Resistors_SMD:R_0805_HandSoldering, F.Cu at (187.0, 137.6)
- added R319: 1k, Resistors_SMD:R_0805_HandSoldering, F.Cu at (175.3, 146.2)
- added R320: 10k, Resistors_SMD:R_0805_HandSoldering, F.Cu at (181.6, 139.9)
- added R321: 100, Resistors_SMD:R_0805_HandSoldering, F.Cu at (192.7, 127.8)
- added U101: LM1117, TO_SOT_Packages_SMD:TO-252-2Lead, F.Cu at (221.6, 89.6)
- added U102: AOZ8904, TO_SOT_Packages_SMD:SOT-23-6_Handsoldering, F.Cu at (221.4, 95.5)
- added U103: STM32F103C8Tx, Housings_QFP:LQFP-48_7x7mm_Pitch0.5mm, F.Cu at (150.9, 82.3)
- added U104: LM258W, Power_Integrations:SO-8, F.Cu at (228.6, 95.1)
- added U201: INA219-SOT23, smd-semi:SOT-23-8, F.Cu at (126.5, 62.0)
- added U202: LM324, SMD_Packages:SOIC-14_N, F.Cu at (153.5, 57.9)
- added U203: LT3083, TO_SOT_Packages_THT:Pentawatt_Neutral_Staggered_Verical_TO220-5-T05D, F.Cu at (113.3, 60.5)
- added U204: LM334Z/NOPB, TO_SOT_Packages_THT:TO-92_Inline_Narrow_Oval, F.Cu at (136.1, 75.2)
- added U301: INA219-SOT23, smd-semi:SOT-23-8, F.Cu at (147.9, 144.0)
- added U302: LM324, SMD_Packages:SOIC-14_N, F.Cu at (165.6, 127.6)
- added U303: LT3083, TO_SOT_Packages_THT:Pentawatt_Neutral_Staggered_Verical_TO220-5-T05D, F.Cu at (137.5, 140.6)
- added U304: LM334Z/NOPB, TO_SOT_Packages_THT:TO-92_Inline_Narrow_Oval, F.Cu at (148.9, 139.8)
- added Y101: 8mhz, Crystals:Crystal_HC49-U_Vertical, F.Cu at (252.9, 77.4)

Commit message: Partially routed one channel.
Parts:
- C208: moved to F.Cu
- D201: footprint TO_SOT_Packages_SMD:SOT-23_Handsoldering -> Diodes_SMD:SOD-323; moved to B.Cu
- D301: footprint TO_SOT_Packages_SMD:SOT-23_Handsoldering -> Diodes_SMD:SOD-323
- moved R215 63.1 mm to (149.9, 67.1)
- moved CON101 41.2 mm to (105.2, 86.4)
- moved K301 37.2 mm to (133.1, 116.3)
- moved R208 29.9 mm to (160.0, 66.5), turned to 0 degrees
- moved D201 27.5 mm to (139.2, 47.2), turned to 270 degrees
- moved C203 23.6 mm to (160.0, 70.6)
- moved R202 22.2 mm to (129.3, 59.9), turned to 90 degrees
- moved Q202 21.8 mm to (149.9, 72.1), turned to 180 degrees
- moved R204 20.0 mm to (160.0, 68.6)
- moved Q203 19.6 mm to (144.3, 64.0), turned to 90 degrees
- moved R212 19.2 mm to (162.6, 57.9), turned to 270 degrees
- moved R213 19.1 mm to (164.6, 57.9), turned to 270 degrees
- moved R214 16.8 mm to (149.4, 56.9), turned to 90 degrees
- moved R209 16.8 mm to (156.2, 50.8), turned to 180 degrees
- moved R210 16.8 mm to (156.2, 48.8), turned to 180 degrees
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Connections:
- U202 pad 1: Net-(R212-Pad2) -> /C1-I-SENSE
- U202 pad 10: Net-(R209-Pad1) -> Net-(C204-Pad1)
- U202 pad 12: Net-(C204-Pad1) -> Net-(C205-Pad1)
- U202 pad 13: Net-(R211-Pad1) -> /C1-I-SENSE
- U202 pad 14: Net-(R217-Pad2) -> Net-(R215-Pad2)
- U202 pad 2: Net-(R212-Pad2) -> Net-(R212-Pad1)
- U202 pad 3: /Channel1/12v-AS -> Net-(R209-Pad1)
- U202 pad 5: Net-(C205-Pad1) -> /Channel1/12v-AS
- U202 pad 6: /C1-I-SENSE -> Net-(R212-Pad2)
- U202 pad 7: Net-(R215-Pad2) -> Net-(R212-Pad2)
- U202 pad 8: /C1-I-SENSE -> Net-(R217-Pad2)
- U202 pad 9: Net-(R212-Pad1) -> Net-(R211-Pad1)
Routing:
- net +12V: track 0.00 -> 86.8 mm
- net /Channel1/REG-OUT: track 0.00 -> 61.5 mm
- net /Channel1/12v-AS: track 0.00 -> 51.3 mm, vias 0 -> 2
- net Net-(C208-Pad2): track 0.00 -> 48.9 mm, vias 0 -> 2
- net Net-(R215-Pad2): track 0.00 -> 22.2 mm
- net /C1-I-SENSE: track 0.00 -> 17.4 mm
- net Net-(R211-Pad1): track 0.00 -> 13.5 mm
- net Net-(R212-Pad2): track 0.00 -> 12.5 mm
- net Net-(Q201-Pad3): track 0.00 -> 10.7 mm
- net Net-(R212-Pad1): track 0.00 -> 8.53 mm
- net Net-(C205-Pad1): track 0.00 -> 6.66 mm
- net Net-(C204-Pad1): track 0.00 -> 6.06 mm
- net Net-(R209-Pad1): track 0.00 -> 5.97 mm
- net Net-(R217-Pad2): track 0.00 -> 5.68 mm
- net Net-(R221-Pad1): track 0.00 -> 4.68 mm
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
Commit message: More layout work.
Parts:
- C101: footprint Capacitors_SMD:C_0805_HandSoldering -> gl:C_0805_HandSoldering
- C102, C103, C104: footprint Capacitors_SMD:C_0805_HandSoldering -> gl:C_0805_HandSoldering; moved to B.Cu
- C105, C106, C107, C108, C109, C307: footprint Capacitors_SMD:C_0805 -> gl:C_0805_HandSoldering; moved to B.Cu
- C110, C111, C201, C202, C203, C204, C205, C206, C207, C208, C209, C301, C302, C303, C304, C305, C306, C308, C309: footprint Capacitors_SMD:C_0805 -> gl:C_0805_HandSoldering
- D201: moved to F.Cu
- P101: value CONN_01X02 -> PB1
- P102: value CONN_01X03 -> ENC1
- P103: value CONN_01X02 -> PB2
- P104: value CONN_01X03 -> ENC2
- P105: value CONN_01X02 -> PB3
- P109: value CONN_01X06 -> SWD
- P110: value CONN_01X02 -> CH2_OUT
- P111: value CONN_01X02 -> CH1_OUT
- R101, R102: footprint Resistors_SMD:R_0805_HandSoldering -> gl:R_0805_HandSoldering; moved to B.Cu
- R103, R104, R105, R106, R107, R108, R109, R201, R202, R203, R204, R207, R208, R209, R210, R211, R212, R213, R214, R215, R216, R217, R218, R219, R220, R221, R301, R302, R303, R304, R307, R308, R309, R310, R311, R312, R313, R314, R315, R316, R317, R318, R319, R320, R321: footprint Resistors_SMD:R_0805_HandSoldering -> gl:R_0805_HandSoldering
- R205, R206, R305, R306: footprint Resistors_SMD:R_2512_HandSoldering -> gl:R_2512_HandSoldering
- U101: moved to B.Cu
- moved R108 149.4 mm to (138.7, 82.8), turned to 180 degrees
- moved C111 141.2 mm to (145.3, 98.0)
- moved R104 137.9 mm to (144.3, 81.8), turned to 180 degrees
- moved R107 137.4 mm to (138.7, 93.0), turned to 180 degrees
- moved R106 137.1 mm to (138.7, 80.8)
- moved R101 136.9 mm to (144.3, 78.8), turned to 180 degrees
- moved R105 125.8 mm to (142.7, 96.0)
- moved R109 119.8 mm to (138.7, 90.9)
- moved C110 118.5 mm to (140.2, 98.0), turned to 180 degrees
- moved R102 118.1 mm to (144.3, 76.8)
- moved Y101 113.8 mm to (141.7, 101.6)
- moved P101 111.7 mm to (174.8, 110.7)
- moved P107 95.2 mm to (170.2, 76.2), turned to 180 degrees
- moved U104 90.3 mm to (138.7, 86.9), turned to 270 degrees
- moved C107 89.9 mm to (187.5, 81.5)
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Connections:
- net Net-(C208-Pad2) renamed /Channel1/SET
- net Net-(C308-Pad2) renamed /Channel2/SET
- U103 pad 11: /C2-I-SENSE -> Net-(U103-Pad11)
- U103 pad 13: /C2-V-SENSE -> /CH2_PWR
- U103 pad 14: /LCD1_CS -> /C2-V-SENSE
- U103 pad 15: /SPI_SCK -> /LCD1_MD
- U103 pad 16: /LCD2_CS -> /C2-V-PWM
- U103 pad 17: /SPI_MOSI -> /C2-I-PWM
- U103 pad 18: /CH1_PWR -> /LCD2_CS
- U103 pad 19: /CH2_PWR -> /LCD2_MD
- U103 pad 21: /C2-I-PWM -> /C2-I-SENSE
- U103 pad 22: /C1-I-PWM -> /LCD1_CS
- U103 pad 26: Net-(U103-Pad26) -> /SPI_SCK
- U103 pad 28: /C1-I-LMT -> /SPI_MOSI
- U103 pad 38: /C2-V-PWM -> /C1-I-PWM
- U103 pad 40: /LCD1_MD -> /C1-I-LMT
- U103 pad 41: /LCD2_MD -> /CH1_PWR
- U302 pad 10: Net-(R309-Pad1) -> Net-(C305-Pad1)
- U302 pad 5: Net-(C305-Pad1) -> Net-(R309-Pad1)
- U302 pad 6: /C2-I-SENSE -> Net-(R312-Pad1)
- U302 pad 7: Net-(R315-Pad2) -> /C2-I-SENSE
- U302 pad 8: /C2-I-SENSE -> Net-(R315-Pad2)
- U302 pad 9: Net-(R312-Pad1) -> /C2-I-SENSE
Routing:
- net +12V: track 86.8 -> 204.6 mm
- net /Channel2/12v-AS: track 0.00 -> 55.2 mm, vias 0 -> 2
- net /Channel2/OUT: track 0.00 -> 54.0 mm, vias 0 -> 4
- net /Channel2/SET: track 0.00 -> 54.0 mm, vias 0 -> 2
- net /Channel1/OUT: track 0.00 -> 43.7 mm, vias 0 -> 4
- net /C2-I-SENSE: track 0.00 -> 41.2 mm
- net SDA: track 0.00 -> 39.1 mm, vias 0 -> 4
- net /Channel2/REG-OUT: track 0.00 -> 35.6 mm
- net /C1-I-SENSE: track 17.4 -> 52.7 mm
- net Net-(D201-Pad2): track 0.00 -> 28.9 mm, vias 0 -> 4
- net SCL: track 0.00 -> 24.2 mm, vias 0 -> 4
- net Net-(R315-Pad2): track 0.00 -> 21.1 mm, vias 0 -> 2
- net /C2-I-PWM: track 0.00 -> 19.6 mm
- net Net-(C111-Pad2): track 0.00 -> 19.5 mm, vias 0 -> 2
- net /C2-V-PWM: track 0.00 -> 18.6 mm
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